File: badge.kicad_pcb (KiCad board)
At the start: 2 copper layers, 39.7 x 52.3 mm, 5 parts, among them U1 NT3H2111W0FHKH

Commit message: s
Parts:
- removed ?: , clipboard:6e83f448-3faf-4843-8bed-d94af388a51f
- added L1: L, Library:nfc-coil, F.Cu at (87.1, 90.7)
Connections:
- U1 pad 1: unconnected-(U1-LA-Pad1) -> Net-(U1-LA)
- U1 pad 8: unconnected-(U1-LB-Pad8) -> Net-(U1-LB)
Routing:
- net Net-(U1-LB): track 0.00 -> 10.6 mm, vias 0 -> 1
- net unconnected-(U1-LB-Pad8): track 5.82 -> 0.00 mm, vias 1 -> 0
- net Net-(U1-LA): track 0.00 -> 3.70 mm
- net (no net): vias 1 -> 0
