File: badge.kicad_sch (KiCad schematic)
At the start: 4 parts, among them U1 NT3H2111W0FHKH

Commit message: s
Parts:
- added L1: L, Library:nfc-coil, symbol Device:L
- U1: footprint XQFN-8_L1.6-W1.6-P0.50-BL_NT3H2111W0FHKH -> footprints:XQFN-8_L1.6-W1.6-P0.50-BL_NT3H2111W0FHKH
Connections:
- net at U1.1 (LA): now also L1.1
- net at U1.8 (LB): now also L1.2
Changed lines of the file:
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@@
+	(wire
+		(pts
+			(xy 111.76 90.17) (xy 111.76 99.06)
+		)
+		(stroke
+			(width 0)
+			(type default)
+		)
+	)
 	(wire
 		(pts
@@
 		(pts
 			(xy 99.06 76.2) (xy 104.14 76.2)
+		)
+		(stroke
+			(width 0)
+			(type default)
+		)
+	)
+	(wire
+		(pts
+			(xy 91.44 90.17) (xy 91.44 99.06)
+		)
+		(stroke
+			(width 0)
+			(type default)
+		)
+	)
+	(wire
+		(pts
+			(xy 104.14 90.17) (xy 91.44 90.17)
 		)
 		(stroke
@@
 			)
 		)
-		(property "Footprint" "XQFN-8_L1.6-W1.6-P0.50-BL_NT3H2111W0FHKH"
+		(property "Footprint" "footprints:XQFN-8_L1.6-W1.6-P0.50-BL_NT3H2111W0FHKH"
 			(at 101.6 114.3 0)
 			(hide yes)
@@
 					(unit 1)
 				)
+			)
+		)
+	)
+	(symbol
+		(lib_id "Device:L")
+		(at 107.95 90.17 270)
+		(mirror x)
+		(unit 1)
+		(body_style 1)
+		(exclude_from_sim no)
+		(in_bom yes)
+		(on_board yes)
+		(in_pos_files yes)
+		(dnp no)
+		(property "Reference" "L1"
+			(at 107.95 85.09 90)
+			(show_name no)
+			(do_not_autoplace no)
+			(effects
+				(font
+					(size 1.27 1.27)
+				)
+			)
+		)
+		(property "Value" "L"
+			(at 107.95 87.63 90)
+			(show_name no)
+			(do_not_autoplace no)
+			(effects
+				(font
+					(size 1.27 1.27)
+				)
+			)
+		)
+		(property "Footprint" "Library:nfc-coil"
+			(at 107.95 90.17 0)
+			(hide yes)
+			(show_name no)
+			(do_not_autoplace no)
+			(effects
+				(font
+					(size 1.27 1.27)
+				)
+			)
+		)
+		(property "Datasheet" ""
+			(at 107.95 90.17 0)
+			(hide yes)
+			(show_name no)
+			(do_not_autoplace no)
+			(effects
+				(font
+					(size 1.27 1.27)
+				)
+			)
+		)
+		(property "Description" "Inductor"
+			(at 107.95 90.17 0)
+			(hide yes)
+			(show_name no)
+			(do_not_autoplace no)
+			(effects
+				(font
+					(size 1.27 1.27)
+				)
+			)
+		)
+		(pin "2"
+		)
+		(pin "1"
+		)
+		(instances
+			(project "badge"
+				(path "/508aa04a-4df0-464c-b3fb-bfce5c8d4f16"
+					(reference "L1")
+					(unit 1)
+				)
